File: minigame.brd (EAGLE design)
At the start: 98.7 x 80 mm, 44 parts, among them J1 AVR_SPI_PRG_6PTH, Q1 MMBT2222A, U1 MCP73831, U2 MIC5219 3.3V, Y1 8MHz

Commit message: Preliminary components placement
Parts:
- moved POWER 91.2 mm to (3.81, 36.8), turned to 180 degrees
- moved LED1 88.1 mm to (91.4, 38.1), turned to 270 degrees
- moved R10 72.6 mm to (77.5, 3.81)
- moved C1 72.0 mm to (63.5, 3.81), flipped to the bottom
- moved C4 71.9 mm to (72.4, 5.08)
- moved C2 71.9 mm to (58.4, 3.81), flipped to the bottom
- moved U1 70.0 mm to (74.9, 10.2)
- moved U2 70.0 mm to (80.0, 10.2)
- moved R9 68.7 mm to (87.6, 17.8)
- moved S1 65.9 mm to (26.7, 11.4), turned to 90 degrees
- moved R1 65.2 mm to (61.0, 11.4)
- moved R12 64.8 mm to (25.4, 25.4)
- moved SG1 64.8 mm to (24.1, 34.3), flipped to the bottom
- moved C3 62.0 mm to (58.4, 20.3), flipped to the bottom, turned to 90 degrees
- moved C5 60.3 mm to (66.0, 25.4), flipped to the bottom
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Connections:
- removed net OLED_3V3: OLED128X64.6
Other:
- board size 98.7 x 80 mm -> 97.5 x 41.9 mm
- board text added: "CHARGE"
- board text added: "RX"
- board text added: "TX"

Commit message: board
Parts:
- added U$3: (no value), SparkFun-Aesthetics:OSHW-LOGO-L
- moved POWER 80.0 mm to (83.8, 36.8), turned to 0 degrees
- moved J1 7.62 mm to (2.54, 35.6)
- moved R10 3.59 mm to (80.0, 6.35), flipped to the bottom, turned to 180 degrees
- moved C4 2.84 mm to (74.9, 6.35), flipped to the bottom
- moved C5 1.27 mm to (64.8, 25.4)
- moved C6 1.27 mm to (64.8, 17.8)
- moved S1 1.27 mm to (25.4, 11.4), turned to 180 degrees
- moved JP1 0.63 mm to (48.3, 4.45)
- flipped C7 to the bottom
- flipped C8 to the bottom
- flipped C9 to the bottom
- turned U$1 to 45 degrees
- flipped U1 to the bottom
- flipped U2 to the bottom
Other:
- board text added: "MicroGame"
- board text added: "Oscar Gonzalez - August 2014"
- board text added: "rev. 1.0"
- board text added: "www.BricoGeek.com"

Commit message: Board placement
Parts:
- moved R13 37.2 mm to (92.1, 8.26), flipped to the bottom, turned to 180 degrees
- moved R14 32.9 mm to (92.1, 10.8), flipped to the bottom, turned to 180 degrees
- moved R11 28.8 mm to (92.1, 13.3), flipped to the bottom, turned to 180 degrees
- moved POWER 6.98 mm to (76.8, 36.8)
- moved R12 5.68 mm to (27.9, 20.3), flipped to the bottom, turned to 270 degrees
- moved LED3 5.43 mm to (86.4, 34.9)
- moved LED2 5.24 mm to (86.4, 36.8)
- moved LED1 5.12 mm to (86.4, 38.7)
- moved Q1 3.24 mm to (27.3, 26.0), flipped to the bottom
- moved S1 2.54 mm to (25.4, 8.89)
- moved C7 1.42 mm to (86.4, 13.3)
- moved C9 1.42 mm to (86.4, 8.26)
- moved C8 1.42 mm to (86.4, 10.8)
- moved R5 0.64 mm to (14.0, 17.1), flipped to the bottom
- moved R8 0.64 mm to (76.2, 21.0), flipped to the bottom
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Other:
- board text added: "3v3"
- board text added: "A"
- board text added: "B"
- board text added: "CLK"
- board text added: "CS"
- board text added: "DATA"
- board text added: "DC"
- board text added: "DOWN"
- board text added: "GND"
- board text added: "ISP"
- board text added: "LEFT"
- board text added: "OFF"
- board text added: "ON"
- board text added: "RIGHT"
- board text added: "RST"
- board text added: "Rechargeable CR2450 3.6V Only!"
- board text added: "UP"
- board text added: "VIN"

Commit message: Added holes and dimensions
Parts:
- added U$2, U$4, U$5, U$6: (no value), SparkFun-Electromechanical:STAND-OFF
- moved J1 3.18 mm to (5.08, 33.7)
Changed lines of the file:
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@@
 <text x="88.265" y="36.195" size="1.27" layer="21" font="vector">TX</text>
 <text x="88.265" y="34.29" size="1.27" layer="21" font="vector">RX</text>
-<text x="2.54" y="3.81" size="2.1844" layer="21" font="vector">MicroGame</text>
-<text x="2.54" y="2.54" size="1.016" layer="21" font="vector">Oscar Gonzalez - August 2014</text>
-<text x="69.215" y="2.54" size="1.778" layer="21" font="vector">www.BricoGeek.com</text>
+<text x="5.08" y="3.81" size="2.1844" layer="21" font="vector">MicroGame</text>
+<text x="5.08" y="2.54" size="1.016" layer="21" font="vector">Oscar Gonzalez - August 2014</text>
+<text x="67.31" y="2.54" size="1.778" layer="21" font="vector">www.BricoGeek.com</text>
 <text x="2.54" y="26.035" size="1.016" layer="1" font="vector" rot="R90">rev. 1.0</text>
 <text x="75.565" y="20.32" size="1.778" layer="21">A</text>
@@
 <text x="53.975" y="33.02" size="1.016" layer="21" rot="R270">VIN</text>
 <text x="56.515" y="33.02" size="1.016" layer="21" rot="R270">GND</text>
+<dimension x1="6.35" y1="20.32" x2="0" y2="20.32" x3="3.175" y3="-3.175" textsize="1.778" layer="20"/>
+<dimension x1="13.97" y1="12.7" x2="0" y2="12.7" x3="6.985" y3="-8.255" textsize="1.778" layer="20"/>
+<dimension x1="13.97" y1="27.94" x2="0" y2="27.94" x3="6.985" y3="46.99" textsize="1.778" layer="20"/>
+<dimension x1="21.59" y1="20.32" x2="0" y2="20.32" x3="10.795" y3="52.705" textsize="1.778" layer="20"/>
+<dimension x1="21.59" y1="20.32" x2="21.59" y2="0" x3="-6.985" y3="10.16" textsize="1.778" layer="20"/>
+<dimension x1="30.48" y1="39.37" x2="0" y2="39.37" x3="15.24" y3="57.785" textsize="1.778" layer="20"/>
+<dimension x1="30.48" y1="39.37" x2="30.48" y2="3.175" x3="-11.43" y3="21.2725" textsize="1.778" layer="20"/>
+<dimension x1="30.48" y1="39.37" x2="66.04" y2="39.37" x3="48.26" y3="57.785" textsize="1.778" layer="20"/>
+<dimension x1="87.63" y1="22.86" x2="97.155" y2="22.86" x3="92.3925" y3="46.355" textsize="1.778" layer="20"/>
+<dimension x1="76.2" y1="16.51" x2="97.155" y2="16.51" x3="86.6775" y3="-3.175" textsize="1.778" layer="20"/>
+<dimension x1="76.2" y1="16.51" x2="76.2" y2="0" x3="104.14" y3="8.255" textsize="1.778" layer="20"/>
+<dimension x1="87.63" y1="22.86" x2="87.63" y2="0" x3="111.76" y3="11.43" textsize="1.778" layer="20"/>
+<dimension x1="0" y1="0" x2="97.46" y2="0" x3="48.73" y3="-15.875" textsize="1.016" layer="20"/>
+<dimension x1="97.46" y1="41.9" x2="97.46" y2="0" x3="118.11" y3="20.95" textsize="1.778" layer="20"/>
+<dimension x1="97.46" y1="41.9" x2="73.025" y2="41.91" x3="85.245878125" y3="50.16" textsize="1.778" layer="20"/>
 </plain>
 <attributes>
@@
 <element name="C2" library="SparkFun-Passives" package="1206" value="22pF" x="58.42" y="3.81" rot="MR0"/>
 <element name="C3" library="SparkFun-Passives" package="1206" value="1uF" x="58.42" y="20.32" rot="MR90"/>
-<element name="J1" library="SparkFun-Connectors" package="2X3" value="AVR_SPI_PRG_6PTH" x="2.54" y="35.56"/>
+<element name="J1" library="SparkFun-Connectors" package="2X3" value="AVR_SPI_PRG_6PTH" x="5.08" y="33.655"/>
 <element name="JP1" library="SparkFun-Connectors" package="USB-MINIB-NOSTOP" value="USB-SMD-NS" x="48.26" y="4.445" rot="MR90"/>
 <element name="LED1" library="SparkFun-LED" package="LED-0603" value="RED" x="86.36" y="38.735" rot="R270"/>
@@
 <element name="R14" library="rcl" package="M0805" value="330" x="92.075" y="10.795" rot="MR180"/>
 <element name="U$3" library="SparkFun-Aesthetics" package="OSHW-LOGO-L" value="" x="4.445" y="11.43"/>
+<element name="U$2" library="SparkFun-Electromechanical" package="STAND-OFF" value="" x="2.54" y="39.37"/>
+<element name="U$4" library="SparkFun-Electromechanical" package="STAND-OFF" value="" x="2.54" y="2.54"/>
+<element name="U$5" library="SparkFun-Electromechanical" package="STAND-OFF" value="" x="94.615" y="2.54"/>
+<element name="U$6" library="SparkFun-Electromechanical" package="STAND-OFF" value="" x="94.615" y="39.37"/>
 </elements>
 <signals>
@@
 <wire x1="7.3" y1="24.765" x2="14.92" y2="17.145" width="0" layer="19" extent="16-16"/>
 <wire x1="13.02" y1="33.02" x2="7.3" y2="24.765" width="0" layer="19" extent="16-16"/>
-<wire x1="7.62" y1="38.1" x2="13.02" y2="33.02" width="0" layer="19" extent="16-16"/>
+<wire x1="10.16" y1="36.195" x2="13.02" y2="33.02" width="0" layer="19" extent="16-16"/>
 <wire x1="28.194" y1="6.985" x2="14.92" y2="17.145" width="0" layer="19" extent="1-16"/>
 </signal>
@@
 <wire x1="17.945" y1="10.45" x2="25.565" y2="18.07" width="0" layer="19" extent="1-1"/>
 <wire x1="10.325" y1="18.07" x2="17.945" y2="25.69" width="0" layer="19" extent="1-1"/>
-<wire x1="2.54" y1="38.1" x2="20.88" y2="34.29" width="0" layer="19" extent="1-1"/>
+<wire x1="5.08" y1="36.195" x2="20.88" y2="34.29" width="0" layer="19" extent="1-1"/>
 </signal>
 <signal name="N$4">
@@
 <contactref element="J1" pad="1"/>
 <contactref element="U$1" pad="11"/>
-<wire x1="2.54" y1="35.56" x2="49.53279375" y2="13.390353125" width="0" layer="19" extent="16-16"/>
+<wire x1="5.08" y1="33.655" x2="49.53279375" y2="13.390353125" width="0" layer="19" extent="16-16"/>
 </signal>
 <signal name="SCK">
 <contactref element="J1" pad="3"/>
 <contactref element="U$1" pad="9"/>
-<wire x1="5.08" y1="35.56" x2="50.664165625" y2="14.521721875" width="0" layer="19" extent="16-16"/>
+<wire x1="7.62" y1="33.655" x2="50.664165625" y2="14.521721875" width="0" layer="19" extent="16-16"/>
 </signal>
 <signal name="RST">
@@
 <wire x1="46.421525" y1="13.9560375" x2="60.01" y2="11.43" width="0" layer="19" extent="16-16"/>
 <wire x1="28.194" y1="10.795" x2="46.421525" y2="13.9560375" width="0" layer="19" extent="1-16"/>
-<wire x1="7.62" y1="35.56" x2="28.194" y2="10.795" width="0" layer="19" extent="1-1"/>
+<wire x1="10.16" y1="33.655" x2="28.194" y2="10.795" width="0" layer="19" extent="1-1"/>
 </signal>
 <signal name="MOSI">
 <contactref element="J1" pad="4"/>
 <contactref element="U$1" pad="10"/>
-<wire x1="5.08" y1="38.1" x2="50.098478125" y2="13.9560375" width="0" layer="19" extent="16-16"/>
+<wire x1="7.62" y1="36.195" x2="50.098478125" y2="13.9560375" width="0" layer="19" extent="16-16"/>
 </signal>
 <signal name="OLED_DATA">

Commit message: Holes fix
Parts:
- moved BAT1 2.54 mm to (80.0, 30.5)
- moved C7 1.91 mm to (86.4, 11.4)
- moved C9 1.91 mm to (86.4, 6.35)
- moved R11 1.91 mm to (92.1, 11.4)
- moved R13 1.91 mm to (92.1, 6.35)
- moved C8 1.90 mm to (86.4, 8.89)
- moved R14 1.90 mm to (92.1, 8.89)
- moved C5 1.90 mm to (62.9, 25.4)
Changed lines of the file:
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@@
 <attribute name="PROD_ID" value="SWCH-11966" x="87.63" y="22.86" size="1.778" layer="27" display="off"/>
 </element>
-<element name="BAT1" library="SparkFun-Electromechanical" package="BATTCON_245MM_PTH" value="3.6V-PRT-10319" x="82.55" y="30.48" rot="MR0"/>
+<element name="BAT1" library="SparkFun-Electromechanical" package="BATTCON_245MM_PTH" value="3.6V-PRT-10319" x="80.01" y="30.48" rot="MR0"/>
 <element name="U1" library="SparkFun-PowerIC" package="SOT23-5" value="MCP73831" x="74.93" y="10.16" rot="MR0">
 <attribute name="PROD_ID" value="IC-09995" x="74.93" y="10.16" size="1.778" layer="28" rot="MR0" display="off"/>
@@
 <element name="R10" library="rcl" package="M0805" value="30k" x="80.01" y="6.35" rot="MR180"/>
 <element name="C4" library="SparkFun-Passives" package="1206" value="4.7uF" x="74.93" y="6.35" rot="MR0"/>
-<element name="C5" library="SparkFun-Capacitors" package="PANASONIC_D" value="10uF" x="64.77" y="25.4" rot="MR0"/>
-<element name="R11" library="rcl" package="M0805" value="470" x="92.075" y="13.335" rot="MR180"/>
+<element name="C5" library="SparkFun-Capacitors" package="PANASONIC_D" value="10uF" x="62.865" y="25.4" rot="MR0"/>
+<element name="R11" library="rcl" package="M0805" value="470" x="92.075" y="11.43" rot="MR180"/>
 <element name="U2" library="SparkFun-PowerIC" package="SOT23-5" value="MIC5219 3.3V" x="80.01" y="10.16" rot="MR0">
 <attribute name="PROD_ID" value="VREG-09872" x="80.01" y="10.16" size="1.778" layer="28" rot="MR0" display="off"/>
 </element>
 <element name="C6" library="SparkFun-Capacitors" package="PANASONIC_D" value="10uF" x="64.77" y="17.78" rot="MR0"/>
-<element name="C7" library="SparkFun-Passives" package="1206" value="470pF" x="86.36" y="13.335" rot="MR0"/>
-<element name="C8" library="SparkFun-Passives" package="1206" value="1uF" x="86.36" y="10.795" rot="MR0"/>
-<element name="C9" library="SparkFun-Passives" package="1206" value="0.1uF" x="86.36" y="8.255" rot="MR0"/>
+<element name="C7" library="SparkFun-Passives" package="1206" value="470pF" x="86.36" y="11.43" rot="MR0"/>
+<element name="C8" library="SparkFun-Passives" package="1206" value="1uF" x="86.36" y="8.89" rot="MR0"/>
+<element name="C9" library="SparkFun-Passives" package="1206" value="0.1uF" x="86.36" y="6.35" rot="MR0"/>
 <element name="SG1" library="SparkFun-Electromechanical" package="BUZZER-12MM" value="BUZZERPTH" x="24.13" y="34.29" rot="MR0"/>
 <element name="Q1" library="SparkFun-DiscreteSemi" package="SOT23-3" value="MMBT2222A" x="27.305" y="26.035" rot="MR0">
@@
 <element name="LED2" library="SparkFun-LED" package="LED-0603" value="YELLOW" x="86.36" y="36.83" rot="R270"/>
 <element name="LED3" library="SparkFun-LED" package="LED-0603" value="BLUE" x="86.36" y="34.925" rot="R270"/>
-<element name="R13" library="rcl" package="M0805" value="330" x="92.075" y="8.255" rot="MR180"/>
-<element name="R14" library="rcl" package="M0805" value="330" x="92.075" y="10.795" rot="MR180"/>
+<element name="R13" library="rcl" package="M0805" value="330" x="92.075" y="6.35" rot="MR180"/>
+<element name="R14" library="rcl" package="M0805" value="330" x="92.075" y="8.89" rot="MR180"/>
 <element name="U$3" library="SparkFun-Aesthetics" package="OSHW-LOGO-L" value="" x="4.445" y="11.43"/>
 <element name="U$2" library="SparkFun-Electromechanical" package="STAND-OFF" value="" x="2.54" y="39.37"/>
@@
 <contactref element="LED3" pad="C"/>
 <wire x1="87.237" y1="34.925" x2="87.237" y2="36.83" width="0" layer="19" extent="1-1"/>
-<wire x1="82.55" y1="30.48" x2="87.237" y2="34.925" width="0" layer="19" extent="1-16"/>
-<wire x1="77.15" y1="20.955" x2="82.55" y2="30.48" width="0" layer="19" extent="16-16"/>
+<wire x1="80.01" y1="30.48" x2="87.237" y2="34.925" width="0" layer="19" extent="1-16"/>
+<wire x1="77.15" y1="20.955" x2="80.01" y2="30.48" width="0" layer="19" extent="16-16"/>
 <wire x1="67.17" y1="17.78" x2="77.15" y2="20.955" width="0" layer="19" extent="16-16"/>
-<wire x1="67.17" y1="25.4" x2="67.17" y2="17.78" width="0" layer="19" extent="16-16"/>
+<wire x1="65.265" y1="25.4" x2="67.17" y2="17.78" width="0" layer="19" extent="16-16"/>
 <wire x1="58.42" y1="18.92" x2="67.17" y2="17.78" width="0" layer="19" extent="16-16"/>
 <wire x1="54.6239625" y1="22.158475" x2="58.42" y2="18.92" width="0" layer="19" extent="16-16"/>
@@
 <wire x1="57.15" y1="35.56" x2="50.098478125" y2="26.683959375" width="0" layer="19" extent="16-16"/>
 <wire x1="88.58" y1="18.415" x2="77.15" y2="20.955" width="0" layer="19" extent="16-16"/>
-<wire x1="87.76" y1="13.335" x2="88.58" y2="18.415" width="0" layer="19" extent="16-16"/>
-<wire x1="87.76" y1="10.795" x2="87.76" y2="13.335" width="0" layer="19" extent="16-16"/>
-<wire x1="87.76" y1="8.255" x2="87.76" y2="10.795" width="0" layer="19" extent="16-16"/>
-<wire x1="80.96" y1="6.35" x2="87.76" y2="8.255" width="0" layer="19" extent="16-16"/>
+<wire x1="87.76" y1="11.43" x2="88.58" y2="18.415" width="0" layer="19" extent="16-16"/>
+<wire x1="87.76" y1="8.89" x2="87.76" y2="11.43" width="0" layer="19" extent="16-16"/>
+<wire x1="87.76" y1="6.35" x2="87.76" y2="8.89" width="0" layer="19" extent="16-16"/>
+<wire x1="80.96" y1="6.35" x2="87.76" y2="6.35" width="0" layer="19" extent="16-16"/>
 <wire x1="80.01" y1="8.8599" x2="80.96" y2="6.35" width="0" layer="19" extent="16-16"/>
 <wire x1="76.33" y1="6.35" x2="80.01" y2="8.8599" width="0" layer="19" extent="16-16"/>
@@
 <contactref element="OLED128X64" pad="7"/>
 <contactref element="SG1" pad="+"/>
-<wire x1="84.96" y1="10.795" x2="91.605" y2="20.61" width="0" layer="19" extent="1-16"/>
-<wire x1="84.96" y1="8.255" x2="84.96" y2="10.795" width="0" layer="19" extent="16-16"/>
-<wire x1="80.96" y1="11.4601" x2="84.96" y2="10.795" width="0" layer="19" extent="16-16"/>
+<wire x1="84.96" y1="8.89" x2="91.605" y2="20.61" width="0" layer="19" extent="1-16"/>
+<wire x1="84.96" y1="6.35" x2="84.96" y2="8.89" width="0" layer="19" extent="16-16"/>
+<wire x1="80.96" y1="11.4601" x2="84.96" y2="8.89" width="0" layer="19" extent="16-16"/>
 <wire x1="80.175" y1="14.26" x2="80.96" y2="11.4601" width="0" layer="19" extent="1-16"/>
 <wire x1="62.37" y1="17.78" x2="80.175" y2="14.26" width="0" layer="19" extent="1-16"/>
@@
 <contactref element="R11" pad="1"/>
 <contactref element="U$1" pad="28"/>
-<wire x1="75.88" y1="8.8599" x2="91.125" y2="13.335" width="0" layer="19" extent="16-16"/>
+<wire x1="75.88" y1="8.8599" x2="91.125" y2="11.43" width="0" layer="19" extent="16-16"/>
 <wire x1="44.15878125" y1="24.42121875" x2="75.88" y2="8.8599" width="0" layer="19" extent="16-16"/>
 </signal>
@@
 <contactref element="LED1" pad="C"/>
 <contactref element="R11" pad="2"/>
-<wire x1="93.025" y1="13.335" x2="87.237" y2="38.735" width="0" layer="19" extent="1-16"/>
+<wire x1="93.025" y1="11.43" x2="87.237" y2="38.735" width="0" layer="19" extent="1-16"/>
 </signal>
 <signal name="N$10">
@@
 <contactref element="U2" pad="4"/>
 <contactref element="C7" pad="2"/>
-<wire x1="79.06" y1="11.4601" x2="84.96" y2="13.335" width="0" layer="19" extent="16-16"/>
+<wire x1="79.06" y1="11.4601" x2="84.96" y2="11.43" width="0" layer="19" extent="16-16"/>
 </signal>
 <signal name="VBAT">
@@
 <contactref element="POWER" pad="2"/>
 <contactref element="BAT1" pad="3"/>
-<wire x1="69.85" y1="30.48" x2="76.835" y2="39.655" width="0" layer="19" extent="1-1"/>
-<wire x1="62.37" y1="25.4" x2="69.85" y2="30.48" width="0" layer="19" extent="16-16"/>
-<wire x1="73.98" y1="8.8599" x2="62.37" y2="25.4" width="0" layer="19" extent="16-16"/>
+<wire x1="67.31" y1="30.48" x2="76.835" y2="39.655" width="0" layer="19" extent="1-1"/>
+<wire x1="60.465" y1="25.4" x2="67.31" y2="30.48" width="0" layer="19" extent="16-16"/>
+<wire x1="73.98" y1="8.8599" x2="60.465" y2="25.4" width="0" layer="19" extent="16-16"/>
 </signal>
 <signal name="N$3">
@@
 <contactref element="R13" pad="2"/>
 <contactref element="LED2" pad="A"/>
-<wire x1="93.025" y1="8.255" x2="85.483" y2="36.83" width="0" layer="19" extent="1-16"/>
+<wire x1="93.025" y1="6.35" x2="85.483" y2="36.83" width="0" layer="19" extent="1-16"/>
 </signal>
 <signal name="N$13">
 <contactref element="R14" pad="2"/>
 <contactref element="LED3" pad="A"/>
-<wire x1="93.025" y1="10.795" x2="85.483" y2="34.925" width="0" layer="19" extent="1-16"/>
+<wire x1="93.025" y1="8.89" x2="85.483" y2="34.925" width="0" layer="19" extent="1-16"/>
 </signal>
 <signal name="N$15">
 <contactref element="U$1" pad="22"/>
 <contactref element="R13" pad="1"/>
-<wire x1="41.33035625" y1="19.04720625" x2="91.125" y2="8.255" width="0" layer="19" extent="16-16"/>
+<wire x1="41.33035625" y1="19.04720625" x2="91.125" y2="6.35" width="0" layer="19" extent="16-16"/>
 </signal>
 <signal name="N$16">
 <contactref element="U$1" pad="8"/>
 <contactref element="R14" pad="1"/>
-<wire x1="51.22985" y1="15.087409375" x2="91.125" y2="10.795" width="0" layer="19" extent="16-16"/>
+<wire x1="51.22985" y1="15.087409375" x2="91.125" y2="8.89" width="0" layer="19" extent="16-16"/>
 </signal>
 </signals>

Commit message: Ajuste en PCB
Parts:
- moved J1 35.7 mm to (36.2, 16.2), flipped to the bottom, turned to 270 degrees
- moved C6 31.1 mm to (34.9, 26.7)
- moved C5 1.80 mm to (61.6, 26.7)
Other:
- board text added: "RESET"
- board text added: "USB"

Commit message: Ripup board layout
Parts:
- moved R12 12.9 mm to (33.1, 32.1), turned to 0 degrees
- moved Q1 11.9 mm to (33.1, 36.4)
- moved R6 0.30 mm to (6.05, 24.8)
- turned U$1 to 90 degrees
